File: ProcessTestbenchHardware/ProcessTestbenchHardware.kicad_pcb (KiCad board)
At the start: 2 copper layers, 50 parts, among them Q1 IRLZ44N, Q2 IRLZ44N, Q3 IRLZ44N, Q4 IRF540N, Q5 IRLZ44N, Q6 IRLZ44N

Commit message: max485
Parts:
- removed Agitador1: Agitador1, TerminalBlock_Phoenix:TerminalBlock_Phoenix_MKDS-1,5-2-5.08_1x02_P5.08mm_Horizontal
- removed ModuloRS485: ModuloRS485, Connector_PinSocket_2.54mm:PinSocket_1x04_P2.54mm_Vertical
- removed the Q4 at (145.5, 112.5)
- added C7: 100nF, Capacitor_THT:C_Disc_D3.0mm_W1.6mm_P2.50mm, F.Cu at (69.5, 97.0)
- added C8: 100nF, Capacitor_THT:C_Disc_D3.0mm_W1.6mm_P2.50mm, F.Cu at (146.4, 64.0)
- added C9: 100nF, Capacitor_THT:C_Disc_D3.0mm_W1.6mm_P2.50mm, F.Cu at (149.2, 95.5)
- added R13: 560, Resistor_THT:R_Axial_DIN0207_L6.3mm_D2.5mm_P7.62mm_Horizontal, F.Cu at (68.7, 79.5)
- added R14: 270, Resistor_THT:R_Axial_DIN0207_L6.3mm_D2.5mm_P7.62mm_Horizontal, F.Cu at (69.5, 90.8)
- added RS485: RS485, TerminalBlock_Phoenix:TerminalBlock_Phoenix_MKDS-1,5-2-5.08_1x02_P5.08mm_Horizontal, F.Cu at (60.0, 96.4)
- added U2: MAX485E, Package_DIP:DIP-8_W7.62mm, F.Cu at (81.3, 93.3)
- R11: value 1k -> 560
- R12: value 9k1 -> 270
- moved R12 109.4 mm to (62.5, 90.8)
- moved R11 95.1 mm to (76.3, 103.0), turned to 180 degrees
- moved Fluxo1 81.9 mm to (199.8, 43.0), turned to 180 degrees
- moved Q1 79.0 mm to (81.5, 103.0)
- moved Cooler1 78.5 mm to (81.5, 114.0)
- moved Cooler2 78.0 mm to (94.5, 114.0)
- moved Q2 77.5 mm to (94.5, 103.0)
- moved Fluxo3 68.0 mm to (188.0, 113.5)
- moved Fluxo2 67.5 mm to (169.6, 113.5)
- moved C6 56.5 mm to (179.2, 71.8), turned to 0 degrees
- moved C5 48.7 mm to (187.7, 88.8), turned to 180 degrees
- moved Press2 47.0 mm to (146.5, 113.5)
- moved C2 43.5 mm to (187.5, 96.8), turned to 180 degrees
- moved C3 42.4 mm to (186.0, 64.3), turned to 0 degrees
- moved R5 38.5 mm to (144.7, 77.3), turned to 90 degrees
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- renumbered Q5 to Q1, Q6 to Q2, Q1 to Q4, Q2 to Q5
Connections:
- A1 pad 10: /Agitador -> /DE/RE_MAX485
- AD620_1 pad 5: Net-(AD620_1-Ref) -> /AD620Ref
- AD620_2 pad 5: Net-(AD620_2-Ref) -> /AD620Ref
- DimmerControlPins1 pad 2: /DimmerControl -> /ZcDimmer
- DimmerControlPins1 pad 3: /ZcDimmer -> /DimmerControl
- PowerSuply1 pad 1: +12V -> GND
- PowerSuply1 pad 2: GND -> +12V
- Q1 pad 1: /cooler -> /Cooler
- Q2 pad 1: /cooler -> /Cooler
- R10 pad 1: Net-(AD620_1-Ref) -> /AD620Ref
- R11 pad 1: GND -> +5V
- R11 pad 2: Net-(AD620_2-Ref) -> Net-(RS485-Pin_2)
- R12 pad 1: Net-(AD620_2-Ref) -> Net-(RS485-Pin_2)
- R12 pad 2: +5V -> Net-(RS485-Pin_1)
- R9 pad 2: Net-(AD620_1-Ref) -> /AD620Ref
Routing:
- net +5V: track 0.00 -> 349.9 mm
- net +12V: track 0.00 -> 191.9 mm
- net GND: track 0.00 -> 15.3 mm
- net /AnalogTemp2: track 0.00 -> 10.3 mm
- net /AnalogTemp1: track 0.00 -> 0.77 mm

Commit message: PinHeadersForSensorsConnections
Parts:
- removed Fluxo1: Fluxo1, TerminalBlock_Phoenix:TerminalBlock_Phoenix_MKDS-1,5-3-5.08_1x03_P5.08mm_Horizontal
- removed Fluxo2: Fluxo2, TerminalBlock_Phoenix:TerminalBlock_Phoenix_MKDS-1,5-3-5.08_1x03_P5.08mm_Horizontal
- removed Fluxo3: Fluxo3, TerminalBlock_Phoenix:TerminalBlock_Phoenix_MKDS-1,5-3-5.08_1x03_P5.08mm_Horizontal
- removed LSHH1: LSHH1, TerminalBlock_Phoenix:TerminalBlock_Phoenix_MKDS-1,5-2-5.08_1x02_P5.08mm_Horizontal
- removed LSHH2: LSHH2, TerminalBlock_Phoenix:TerminalBlock_Phoenix_MKDS-1,5-2-5.08_1x02_P5.08mm_Horizontal
- removed LSLL1: LSLL1, TerminalBlock_Phoenix:TerminalBlock_Phoenix_MKDS-1,5-2-5.08_1x02_P5.08mm_Horizontal
- removed LSLL2: LSLL2, TerminalBlock_Phoenix:TerminalBlock_Phoenix_MKDS-1,5-2-5.08_1x02_P5.08mm_Horizontal
- removed Press1, Press2: Press1, TerminalBlock_Phoenix:TerminalBlock_Phoenix_MKDS-1,5-4-5.08_1x04_P5.08mm_Horizontal
- removed Term1: Term1, TerminalBlock_Phoenix:TerminalBlock_Phoenix_MKDS-1,5-2-5.08_1x02_P5.08mm_Horizontal
- removed Term2: Term2, TerminalBlock_Phoenix:TerminalBlock_Phoenix_MKDS-1,5-2-5.08_1x02_P5.08mm_Horizontal
- added J1: Fluxo1, Connector_PinHeader_2.54mm:PinHeader_1x03_P2.54mm_Horizontal, F.Cu at (153.4, 81.7)
- added J11: LSLL1, Connector_PinHeader_2.54mm:PinHeader_1x02_P2.54mm_Horizontal, F.Cu at (97.4, 57.3)
- added J12: LSHH2, Connector_PinHeader_2.54mm:PinHeader_1x02_P2.54mm_Horizontal, F.Cu at (88.4, 57.3)
- added J13: LSLL2, Connector_PinHeader_2.54mm:PinHeader_1x02_P2.54mm_Horizontal, F.Cu at (79.4, 57.4)
- added J2: Fluxo2, Connector_PinHeader_2.54mm:PinHeader_1x03_P2.54mm_Horizontal, F.Cu at (153.8, 105.5)
- added J3: Fluxo, Connector_PinHeader_2.54mm:PinHeader_1x03_P2.54mm_Horizontal, F.Cu at (142.0, 105.5)
- added J4: Pressao1, Connector_PinHeader_2.54mm:PinHeader_1x04_P2.54mm_Horizontal, F.Cu at (115.4, 57.4)
- added J5: Pressao2, Connector_PinHeader_2.54mm:PinHeader_1x04_P2.54mm_Horizontal, F.Cu at (153.5, 92.9)
- added J6: Term1, Connector_PinHeader_2.54mm:PinHeader_1x02_P2.54mm_Horizontal, F.Cu at (69.9, 57.3)
- added J7: Term2, Connector_PinHeader_2.54mm:PinHeader_1x02_P2.54mm_Horizontal, F.Cu at (60.9, 57.3)
- added J8: LSHH1, Connector_PinHeader_2.54mm:PinHeader_1x02_P2.54mm_Horizontal, F.Cu at (106.4, 57.3)
- moved RS485 97.1 mm to (154.7, 75.0), turned to 90 degrees
- moved C7 82.0 mm to (143.8, 62.2)
- moved R14 80.0 mm to (149.0, 81.9), turned to -90 degrees
- moved R11 77.1 mm to (138.2, 57.0), turned to 0 degrees
- moved R12 76.2 mm to (132.9, 61.8), turned to 0 degrees
- moved U2 75.1 mm to (150.7, 64.6), turned to 90 degrees
- moved R13 63.1 mm to (127.7, 57.0)
- moved C5 56.8 mm to (131.0, 91.8), turned to 90 degrees
- moved C4 56.4 mm to (131.0, 86.5), turned to 90 degrees
- moved R4 53.8 mm to (98.2, 61.9)
- moved C6 53.3 mm to (131.0, 94.5), turned to -90 degrees
- moved LM358 53.2 mm to (103.0, 69.5)
- moved R9 53.2 mm to (115.0, 69.6), turned to 90 degrees
- moved C3 48.4 mm to (147.5, 93.8), turned to -90 degrees
- moved R3 46.8 mm to (93.5, 61.9)
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Routing:
- net +5V: track 349.9 -> 0.00 mm
- net +12V: track 191.9 -> 5.01 mm
- net GND: track 15.3 -> 0.00 mm
- net /AnalogTemp2: track 10.3 -> 0.00 mm
- net /AnalogTemp1: track 0.77 -> 0.00 mm
Other:
- board outline added: 104 x 63 mm

Commit message: PCB routing
Parts:
- added J14: Servo, Connector_PinHeader_2.54mm:PinHeader_1x03_P2.54mm_Horizontal, F.Cu at (153.5, 106.4)
- J3: value Fluxo -> Fluxo3
- moved J2 13.2 mm to (140.6, 105.5)
- moved R7 7.68 mm to (83.5, 69.6), turned to 90 degrees
- moved R12 7.62 mm to (140.6, 61.8), turned to 180 degrees
- moved J3 7.50 mm to (149.5, 105.4)
- moved C8 2.50 mm to (131.0, 76.0), turned to 90 degrees
Routing:
- net +5V: track 0.00 -> 333.3 mm, vias 0 -> 2
- net /MAX485_RX: track 0.00 -> 158.4 mm, vias 0 -> 3
- net /MAX485_TX: track 0.00 -> 139.7 mm, vias 0 -> 2
- net +12V: track 5.01 -> 132.9 mm, vias 0 -> 1
- net /DE/RE_MAX485: track 0.00 -> 126.1 mm, vias 0 -> 2
- net -5V: track 0.00 -> 87.8 mm, vias 0 -> 1
- net /SaidaServoMotor: track 0.00 -> 82.8 mm, vias 0 -> 3
- net Net-(RS485-Pin_1): track 0.00 -> 77.9 mm, vias 0 -> 3
- net /AnalogTemp2: track 0.00 -> 60.8 mm, vias 0 -> 2
- net /AnalogTemp1: track 0.00 -> 51.7 mm, vias 0 -> 1
- net /AD620Ref: track 0.00 -> 48.5 mm, vias 0 -> 1
- net /LSLL2: track 0.00 -> 48.1 mm, vias 0 -> 1
- net Net-(LM358B-+): track 0.00 -> 47.1 mm, vias 0 -> 3
- net /DimmerControl: track 0.00 -> 46.0 mm
- net Net-(RS485-Pin_2): track 0.00 -> 43.6 mm
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- added copper zone on B.Cu, net GND
Other:
- board size 104 x 63 mm -> 107 x 70 mm
