File: ProcessTestbenchHardware/ProcessTestbenchHardware.kicad_sch (KiCad schematic)
At the start: 53 parts, among them J1 Screw_Terminal_01x02, J10 Screw_Terminal_01x02, J2 ModuloRS485, J8 DB15, J9 Screw_Terminal_01x02, Q1 IRLZ44N, Q2 IRLZ44N, Q3 IRLZ44N, Q4 IRF540N, Q5 IRLZ44N, Q6 IRLZ44N, SW6 LSLL1, SW7 LSHH1, U3 ICL7660, U4 AD620, U5 AD620, U6 LM358, U7 LM358

Commit message: FootprintsAdded
Parts:
- removed SW6: LSLL1, symbol Switch:SW_SPST
- removed SW7: LSHH1, symbol Switch:SW_SPST
- added LSHH1, LSLL1: Screw_Terminal_01x02, TerminalBlock:TerminalBlock_MaiXu_MX126-5.0-02P_1x02_P5.00mm, symbol Connector:Screw_Terminal_01x02
- Agitador1: renamed from Agitador; footprint (none) -> TerminalBlock:TerminalBlock_MaiXu_MX126-5.0-02P_1x02_P5.00mm
- Bomba1, Bomba2, Cooler1, Cooler2, J1, J10, J9, LSHH2, LSLL2, Term1, Term2: footprint (none) -> TerminalBlock:TerminalBlock_MaiXu_MX126-5.0-02P_1x02_P5.00mm
- C1, C2, C3: footprint (none) -> Capacitor_THT:CP_Radial_D4.0mm_P1.50mm
- C4, C5, C6: footprint (none) -> Capacitor_THT:C_Disc_D3.0mm_W1.6mm_P2.50mm
- Fluxo2, Fluxo3: footprint (none) -> TerminalBlock:TerminalBlock_MaiXu_MX126-5.0-03P_1x03_P5.00mm
- J2: footprint (none) -> Connector_PinSocket_1.00mm:PinSocket_1x04_P1.00mm_Vertical
- J8: footprint (none) -> Connector_Dsub:DSUB-15-HD_Pins_Horizontal_P2.29x2.54mm_EdgePinOffset8.35mm_Housed_MountingHolesOffset10.89mm
- Peltier1: renamed from Peltier; footprint (none) -> TerminalBlock:TerminalBlock_MaiXu_MX126-5.0-02P_1x02_P5.00mm
- Press1, Press2: footprint (none) -> TerminalBlock:TerminalBlock_MaiXu_MX126-5.0-04P_1x04_P5.00mm
- R1, R10, R11, R12, R2, R3, R4, R5, R6, R7, R8, R9: footprint (none) -> Resistor_THT:R_Axial_DIN0204_L3.6mm_D1.6mm_P5.08mm_Horizontal
- U1: now left out of the parts list
- U2: value (none) -> StepDownConverter; footprint (none) -> AddOnsLibrary:StepDownFootprint
- U3, U4, U5, U6: footprint (none) -> Package_DIP:DIP-8_W7.62mm
- U6: renamed from U7; footprint (none) -> Package_DIP:DIP-8_W7.62mm
Connections:
- net +5V: now also LSHH1.1 (Pin_1), LSLL1.1 (Pin_1)
- net AnalogNivel2: now also U6.6 (-), U6.7; no longer U6.1, U6.2 (-)
- net LSHH1: now also LSHH1.2 (Pin_2)
- net LSLL1: now also LSLL1.2 (Pin_2)
- net at U5.6: now also U6.5 (+); no longer U6.3 (+)

Commit message: ScrewTerminalsForDimmer
Parts:
- added Fluxo1: Screw_Terminal_01x03, TerminalBlock:TerminalBlock_MaiXu_MX126-5.0-03P_1x03_P5.00mm, symbol Connector:Screw_Terminal_01x03
- added J3: DimmerControlPins, TerminalBlock:TerminalBlock_MaiXu_MX126-5.0-04P_1x04_P5.00mm, symbol Connector:Screw_Terminal_01x04
- added J4: DimmerControlPins, symbol Connector:Screw_Terminal_01x02
- added unit 3 of U6
- Agitador1: value Screw_Terminal_01x02 -> Agitador1
- Bomba1: value Screw_Terminal_01x02 -> Bomba1
- Bomba2: value Screw_Terminal_01x02 -> Bomba2
- Cooler1: value Screw_Terminal_01x02 -> Cooler1
- Cooler2: value Screw_Terminal_01x02 -> Cooler2
- J10: value Screw_Terminal_01x02 -> LOAD; now left out of the parts list
- J8: symbol Connector:DE15_Pins_HighDensity -> Connector:DE15_Pins_HighDensity_MountingHoles; now not fitted; now left out of the parts list
- J9: value Screw_Terminal_01x02 -> AC In; now left out of the parts list
- LSHH1: value Screw_Terminal_01x02 -> LSHH1
- LSHH2: value Screw_Terminal_01x02 -> LSHH2
- LSLL1: value Screw_Terminal_01x02 -> LSLL1
- LSLL2: value Screw_Terminal_01x02 -> LSLL2
- Peltier1: value Screw_Terminal_01x02 -> Peltier1
- Press1, Press2: value Screw_Terminal_01x04 -> Press1
- Term1: value Screw_Terminal_01x02 -> Term1
- Term2: value Screw_Terminal_01x02 -> Term2
- U2: value StepDownConverter -> StepDown; footprint AddOnsLibrary:StepDownFootprint -> AddOnsLibrary:SRT_MPT1584EN_Module
Connections:
- net +12V: now also U2.1 (IN+); no longer U2. (OUT-)
- net +5V: now also U2.3 (OUT+), Fluxo1.1 (Pin_1), J3.1 (Pin_1), U6.8 (V+); no longer U2. (OUT-)
- net -5V: now also U6.4 (V-)
- net AnalogTemp1: no longer R6.2, Term2.1 (Pin_1)
- net AnalogTemp2: now also R6.2, Term2.1 (Pin_1)
- net DimmerControl: now also J3.2 (Pin_2); no longer U1. (LOAD_N)
- net Fluxo1: now also Fluxo1.2 (Pin_2)
- net GND: now also J8.SH, U2.2 (IN-), U2.4 (OUT-), Fluxo1.3 (Pin_3), J3.4 (Pin_4); no longer U2. (OUT-)
- net ZcDimmer: now also J3.3 (Pin_3); no longer U1. (LOAD_N)
- new net: J4.1 (Pin_1), U1. (LOAD_N)
- new net: J4.2 (Pin_2), U1. (LOAD_N)
- no-connect marks 2 -> 3
Other:
- moved on the sheet: Fluxo2, Fluxo3, J10, J2, J9, LSHH1, LSHH2, LSLL1, LSLL2, Press1, Press2, R1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

Commit message: PcbLayoutBegin
Parts:
- Agitador1, Bomba1, Bomba2, Cooler1, Cooler2, LSHH1, LSHH2, LSLL1, LSLL2, Peltier1, Term1, Term2: footprint TerminalBlock:TerminalBlock_MaiXu_MX126-5.0-02P_1x02_P5.00mm -> TerminalBlock_Phoenix:TerminalBlock_Phoenix_MKDS-1,5-2-5.08_1x02_P5.08mm_Horizontal
- C1, C2, C3: footprint Capacitor_THT:CP_Radial_D4.0mm_P1.50mm -> Capacitor_THT:C_Radial_D5.0mm_H7.0mm_P2.00mm
- DimmerControlPins1: renamed from J3; footprint TerminalBlock:TerminalBlock_MaiXu_MX126-5.0-04P_1x04_P5.00mm -> TerminalBlock_Phoenix:TerminalBlock_Phoenix_MKDS-1,5-4-5.08_1x04_P5.08mm_Horizontal
- Fluxo1: value Screw_Terminal_01x03 -> Fluxo1; footprint TerminalBlock:TerminalBlock_MaiXu_MX126-5.0-03P_1x03_P5.00mm -> TerminalBlock_Phoenix:TerminalBlock_Phoenix_MKDS-1,5-3-5.08_1x03_P5.08mm_Horizontal
- Fluxo2: value Screw_Terminal_01x03 -> Fluxo2; footprint TerminalBlock:TerminalBlock_MaiXu_MX126-5.0-03P_1x03_P5.00mm -> TerminalBlock_Phoenix:TerminalBlock_Phoenix_MKDS-1,5-3-5.08_1x03_P5.08mm_Horizontal
- Fluxo3: value Screw_Terminal_01x03 -> Fluxo3; footprint TerminalBlock:TerminalBlock_MaiXu_MX126-5.0-03P_1x03_P5.00mm -> TerminalBlock_Phoenix:TerminalBlock_Phoenix_MKDS-1,5-3-5.08_1x03_P5.08mm_Horizontal
- ModuloRS485: renamed from J2; footprint Connector_PinSocket_1.00mm:PinSocket_1x04_P1.00mm_Vertical -> Connector_PinSocket_2.54mm:PinSocket_1x04_P2.54mm_Vertical
- PowerSuply1: renamed from J1; value Screw_Terminal_01x02 -> PowerSuply; footprint TerminalBlock:TerminalBlock_MaiXu_MX126-5.0-02P_1x02_P5.00mm -> TerminalBlock_Phoenix:TerminalBlock_Phoenix_MKDS-1,5-2-5.08_1x02_P5.08mm_Horizontal
- Press1, Press2: footprint TerminalBlock:TerminalBlock_MaiXu_MX126-5.0-04P_1x04_P5.00mm -> TerminalBlock_Phoenix:TerminalBlock_Phoenix_MKDS-1,5-4-5.08_1x04_P5.08mm_Horizontal
- R1, R10, R11, R12, R2, R3, R4, R5, R6, R7, R8, R9: footprint Resistor_THT:R_Axial_DIN0204_L3.6mm_D1.6mm_P5.08mm_Horizontal -> Resistor_THT:R_Axial_DIN0207_L6.3mm_D2.5mm_P7.62mm_Horizontal
- renumbered U4 to AD620_1, U5 to AD620_2, U3 to ICL7660, U6 to LM358, U2 to StepDown1
Other:
- note removed: "Power Supply"

Commit message: max485
Parts:
- removed Agitador1: Agitador1, TerminalBlock_Phoenix:TerminalBlock_Phoenix_MKDS-1,5-2-5.08_1x02_P5.08mm_Horizontal, symbol Connector:Screw_Terminal_01x02
- removed J4: DimmerControlPins, symbol Connector:Screw_Terminal_01x02
- removed J8: DB15, Connector_Dsub:DSUB-15-HD_Pins_Horizontal_P2.29x2.54mm_EdgePinOffset8.35mm_Housed_MountingHolesOffset10.89mm, symbol Connector:DE15_Pins_HighDensity_MountingHoles
- removed ModuloRS485: ModuloRS485, Connector_PinSocket_2.54mm:PinSocket_1x04_P2.54mm_Vertical, symbol Connector:Conn_01x04_Socket
- removed Q4: IRF540N, Package_TO_SOT_THT:TO-220-3_Vertical, symbol Transistor_FET:IRF540N
- added C7, C8, C9: 100nF, Capacitor_THT:C_Disc_D3.0mm_W1.6mm_P2.50mm, symbol Device:C
- added DimmerControlPins2: DimmerControlPins(Module), TerminalBlock_Phoenix:TerminalBlock_Phoenix_MKDS-1,5-4-5.08_1x04_P5.08mm_Horizontal, symbol Connector:Screw_Terminal_01x04
- added R13: 560, Resistor_THT:R_Axial_DIN0207_L6.3mm_D2.5mm_P7.62mm_Horizontal, symbol Device:R_US
- added R14: 270, Resistor_THT:R_Axial_DIN0207_L6.3mm_D2.5mm_P7.62mm_Horizontal, symbol Device:R_US
- added RS485: RS485, TerminalBlock_Phoenix:TerminalBlock_Phoenix_MKDS-1,5-2-5.08_1x02_P5.08mm_Horizontal, symbol Connector:Screw_Terminal_01x02
- added U2: MAX485E, Package_DIP:DIP-8_W7.62mm, symbol Interface_UART:MAX485E
- R11: value 1k -> 560
- R12: value 9k1 -> 270
- renumbered Q5 to Q1, Q6 to Q2, Q1 to Q4, Q2 to Q5
Connections:
- net cooler is gone; now on net Cooler: Q1.1 (G), Q2.1 (G)
- net +12V: now also PowerSuply1.2 (Pin_2); no longer PowerSuply1.1 (Pin_1)
- net +5V: now also R11.1, C7.2, C8.2, C9.2, U2.8 (VCC); no longer R12.2, U1. (LOAD_N)
- net DimmerControl: now also DimmerControlPins1.3 (Pin_3); no longer DimmerControlPins1.2 (Pin_2)
- net GND: now also PowerSuply1.1 (Pin_1), C7.1, C8.1, C9.1, R13.2, U2.5 (GND); no longer PowerSuply1.2 (Pin_2), R11.1, U1. (LOAD_N)
- net MAX485_RX: now also U2.1 (RO)
- net MAX485_TX: now also U2.4 (DI)
- net ZcDimmer: now also DimmerControlPins1.2 (Pin_2); no longer DimmerControlPins1.3 (Pin_3)
- net at U1. (LOAD_N): now also J9.2 (Pin_2)
- net AD620Ref: now reaches AD620_1.5 (Ref), R10.1, R9.2
- net AD620Ref: now also AD620_2.5 (Ref)
- net at R11.2, R12.1: now also R14.1, RS485.2 (Pin_2), U2.7 (B); no longer AD620_2.5 (Ref)
- net Agitador renamed DE/RE_MAX485
- net DE/RE_MAX485: now also U2.2 (~{RE}), U2.3 (DE)
- new net: DimmerControlPins2.1 (Pin_1), U1. (LOAD_N)
- new net: DimmerControlPins2.2 (Pin_2), U1. (LOAD_N)
- new net: DimmerControlPins2.3 (Pin_3), U1. (LOAD_N)
- new net: DimmerControlPins2.4 (Pin_4), U1. (LOAD_N)
- new net: R12.2, R13.1, R14.2, RS485.1 (Pin_1), U2.6 (A)
- no-connect marks 3 -> 2
Other:
- moved on the sheet: AD620_1, AD620_2, C1, C2, C3, C4, C5, C6, Cooler1, Cooler2, Fluxo1, Fluxo2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

Commit message: PinHeadersForSensorsConnections
Parts:
- removed Fluxo1: Fluxo1, TerminalBlock_Phoenix:TerminalBlock_Phoenix_MKDS-1,5-3-5.08_1x03_P5.08mm_Horizontal, symbol Connector:Screw_Terminal_01x03
- removed Fluxo2: Fluxo2, TerminalBlock_Phoenix:TerminalBlock_Phoenix_MKDS-1,5-3-5.08_1x03_P5.08mm_Horizontal, symbol Connector:Screw_Terminal_01x03
- removed Fluxo3: Fluxo3, TerminalBlock_Phoenix:TerminalBlock_Phoenix_MKDS-1,5-3-5.08_1x03_P5.08mm_Horizontal, symbol Connector:Screw_Terminal_01x03
- removed LSHH1: LSHH1, TerminalBlock_Phoenix:TerminalBlock_Phoenix_MKDS-1,5-2-5.08_1x02_P5.08mm_Horizontal, symbol Connector:Screw_Terminal_01x02
- removed LSHH2: LSHH2, TerminalBlock_Phoenix:TerminalBlock_Phoenix_MKDS-1,5-2-5.08_1x02_P5.08mm_Horizontal, symbol Connector:Screw_Terminal_01x02
- removed LSLL1: LSLL1, TerminalBlock_Phoenix:TerminalBlock_Phoenix_MKDS-1,5-2-5.08_1x02_P5.08mm_Horizontal, symbol Connector:Screw_Terminal_01x02
- removed LSLL2: LSLL2, TerminalBlock_Phoenix:TerminalBlock_Phoenix_MKDS-1,5-2-5.08_1x02_P5.08mm_Horizontal, symbol Connector:Screw_Terminal_01x02
- removed Press1, Press2: Press1, TerminalBlock_Phoenix:TerminalBlock_Phoenix_MKDS-1,5-4-5.08_1x04_P5.08mm_Horizontal, symbol Connector:Screw_Terminal_01x04
- removed Term1: Term1, TerminalBlock_Phoenix:TerminalBlock_Phoenix_MKDS-1,5-2-5.08_1x02_P5.08mm_Horizontal, symbol Connector:Screw_Terminal_01x02
- removed Term2: Term2, TerminalBlock_Phoenix:TerminalBlock_Phoenix_MKDS-1,5-2-5.08_1x02_P5.08mm_Horizontal, symbol Connector:Screw_Terminal_01x02
- added J1: Fluxo1, Connector_PinHeader_2.54mm:PinHeader_1x03_P2.54mm_Horizontal, symbol Connector:Conn_01x03_Pin
- added J11: LSLL1, Connector_PinHeader_2.54mm:PinHeader_1x02_P2.54mm_Horizontal, symbol Connector:Conn_01x02_Pin
- added J12: LSHH2, Connector_PinHeader_2.54mm:PinHeader_1x02_P2.54mm_Horizontal, symbol Connector:Conn_01x02_Pin
- added J13: LSLL2, Connector_PinHeader_2.54mm:PinHeader_1x02_P2.54mm_Horizontal, symbol Connector:Conn_01x02_Pin
- added J2: Fluxo2, Connector_PinHeader_2.54mm:PinHeader_1x03_P2.54mm_Horizontal, symbol Connector:Conn_01x03_Pin
- added J3: Fluxo, Connector_PinHeader_2.54mm:PinHeader_1x03_P2.54mm_Horizontal, symbol Connector:Conn_01x03_Pin
- added J4: Pressao1, Connector_PinHeader_2.54mm:PinHeader_1x04_P2.54mm_Horizontal, symbol Connector:Conn_01x04_Pin
- added J5: Pressao2, Connector_PinHeader_2.54mm:PinHeader_1x04_P2.54mm_Horizontal, symbol Connector:Conn_01x04_Pin
- added J6: Term1, Connector_PinHeader_2.54mm:PinHeader_1x02_P2.54mm_Horizontal, symbol Connector:Conn_01x02_Pin
- added J7: Term2, Connector_PinHeader_2.54mm:PinHeader_1x02_P2.54mm_Horizontal, symbol Connector:Conn_01x02_Pin
- added J8: LSHH1, Connector_PinHeader_2.54mm:PinHeader_1x02_P2.54mm_Horizontal, symbol Connector:Conn_01x02_Pin
Connections:
- net +5V: now also J1.3 (Pin_3), J11.1 (Pin_1), J12.1 (Pin_1), J13.1 (Pin_1), J2.3 (Pin_3), J3.3 (Pin_3), J4.4 (Pin_4), J5.4 (Pin_4), J8.1 (Pin_1)
- net AnalogTemp1: now also J6.1 (Pin_1)
- net AnalogTemp2: now also J7.1 (Pin_1)
- net Fluxo1: now also J1.2 (Pin_2)
- net Fluxo2: now also J2.2 (Pin_2)
- net Fluxo3: now also J3.2 (Pin_2)
- net GND: now also J1.1 (Pin_1), J2.1 (Pin_1), J3.1 (Pin_1), J4.1 (Pin_1), J5.1 (Pin_1), J6.2 (Pin_2), J7.2 (Pin_2)
- net LSHH1: now also J8.2 (Pin_2)
- net LSHH2: now also J12.2 (Pin_2)
- net LSLL1: now also J11.2 (Pin_2)
- net LSLL2: now also J13.2 (Pin_2)
- net Press1+: now also J4.3 (Pin_3)
- net Press1-: now also J4.2 (Pin_2)
- net Press2+: now also J5.3 (Pin_3)
- net Press2-: now also J5.2 (Pin_2)

Commit message: PCB routing
Parts:
- added J14: Servo, Connector_PinHeader_2.54mm:PinHeader_1x03_P2.54mm_Horizontal, symbol Connector:Conn_01x03_Pin
- J3: value Fluxo -> Fluxo3
Connections:
- net +5V: now also J14.1 (Pin_1)
- net GND: now also J14.3 (Pin_3)
- net SaidaServoMotor: now also J14.2 (Pin_2)
Other:
- moved on the sheet: J7, R6
